File: rc2014-mystorm.sch (KiCad schematic (older format))
At the start: 11 parts, among them J1 CONN_02X06, J2 CONN_02X06, J3 CONN_02X06, J4 CONN_02X17, J5 CONN_01X10, P1 RC2014 BUS, U1 74LVC245, U2 74HC245, U3 74HC245, U4 74HC245, U5 74HC245

Commit message: SMT....
Parts:
- removed J4: CONN_02X17, Socket_Strips:Socket_Strip_Angled_2x17_Pitch2.54mm, symbol CONN_02X17
- removed J5: CONN_01X10, symbol CONN_01X10
- removed U5: 74HC245, Housings_DIP:DIP-20_W7.62mm_Socket, symbol 74HC245
- added C1, C2, C3, C4: C, Capacitors_SMD:C_1206_HandSoldering, symbol C
- added J4, J6: CONN_02X06, Pin_Headers:Pin_Header_Straight_2x06_Pitch2.54mm, symbol CONN_02X06
- added J7: CONN_01X06, Pin_Headers:Pin_Header_Straight_1x06_Pitch2.54mm, symbol Conn_01x06
- U1: value 74LVC245 -> SN74LVCC3245A; footprint Housings_DIP:DIP-20_W7.62mm_Socket -> Housings_SOIC:SOIC-24W_7.5x15.4mm_Pitch1.27mm; symbol 74HC245 -> SN74LVCC3245A
- U2, U3, U4: value 74HC245 -> SN74LVCC3245A; footprint Housings_DIP:DIP-20_W7.62mm_Socket -> Housings_SOIC:SOIC-24W_7.5x15.4mm_Pitch1.27mm; symbol 74HC245 -> SN74LVCC3245A
Connections:
- net labels added: +5V, OE
- net labels removed: BUSACK, BUSACKLV, BUSREQ, BUSREQLV, EXTRA_DIR, EXTRA_OE, HALT, HALTLV, NMI, NMILV, RXLV, S1, S1LV, TXLV, WAIT, WAITLV
- wire segments 206 -> 201
- no-connect marks 8 -> 5

Commit message: further SMT WIP
Parts:
- removed J1, J2, J3, J6: CONN_02X06, Pin_Headers:Pin_Header_Straight_2x06_Pitch2.54mm, symbol CONN_02X06
- removed J7: CONN_01X06, Pin_Headers:Pin_Header_Straight_1x06_Pitch2.54mm, symbol Conn_01x06
- added C1, C2: CP_Small, Capacitors_SMD:C_0805_HandSoldering, symbol CP_Small
- added C10, C11, C12, C7, C8, C9: C, Capacitors_SMD:C_0805_HandSoldering, symbol C
- added J1: FPGA connection, Pin_Headers:Pin_Header_Straight_2x20_Pitch2.54mm, symbol Conn_02x20_Odd_Even
- added J3: Conn_01x05, Pin_Headers:Pin_Header_Straight_1x04_Pitch2.54mm, symbol Conn_01x04
- added J4: Conn_01x03, Pin_Headers:Pin_Header_Straight_1x03_Pitch2.54mm, symbol Conn_01x03
- added J5: Conn_01x05, Pin_Headers:Pin_Header_Straight_1x05_Pitch2.54mm, symbol Conn_01x05
- added J6: Extra, Pin_Headers:Pin_Header_Straight_1x08_Pitch2.54mm, symbol Conn_01x08
- added JP1: Ext Power, Pin_Headers:Pin_Header_Straight_1x03_Pitch2.54mm, symbol Jumper_Dual
- added U4: SN74LVCC3245A, Housings_SOIC:SOIC-24W_7.5x15.4mm_Pitch1.27mm, symbol SN74LVCC3245A
- added U6: LM1117-3.3, TO_SOT_Packages_SMD:SOT-223-3_TabPin2, symbol LM1117-3.3
- C3: renamed from C1; footprint Capacitors_SMD:C_1206_HandSoldering -> Capacitors_SMD:C_0805_HandSoldering
- C4: renamed from C2; footprint Capacitors_SMD:C_1206_HandSoldering -> Capacitors_SMD:C_0805_HandSoldering
- C5: renamed from C3; footprint Capacitors_SMD:C_1206_HandSoldering -> Capacitors_SMD:C_0805_HandSoldering
- C6: renamed from C4; footprint Capacitors_SMD:C_1206_HandSoldering -> Capacitors_SMD:C_0805_HandSoldering
- J2: renamed from J4; value CONN_02X06 -> Config; footprint Pin_Headers:Pin_Header_Straight_2x06_Pitch2.54mm -> Pin_Headers:Pin_Header_Straight_2x08_Pitch2.54mm; symbol CONN_02X06 -> Conn_02x08_Odd_Even
- renumbered U4 to U5
Connections:
- net labels added: EX1, EX1LV, EX2, EX2LV, EX3, EX3LV, EX4, EX4LV, EX5, EX5LV, EX6, EX6LV, EX7, EX7LV, EX8, EX8LV, FPGA_VCC, GPIO1, GPIO2, GPIO3, GPIO4, SIG2_DIR, SIG2_OE
- net labels removed: OE, VCC
- wire segments 201 -> 244
Other:
- moved on the sheet: C3, C4, C5, C6, U5

Commit message: WIP
Parts:
- J1: footprint Pin_Headers:Pin_Header_Straight_2x20_Pitch2.54mm -> Connectors_IDC:IDC-Header_2x20_Pitch2.54mm_Straight
Changed lines of the file:
@@
 	1    0    0    -1
 $EndComp
-Text Label 5550 2700 2    60   ~ 0
-FPGA_VCC
 $Comp
 L GND #PWR018
@@
 F 0 "J1" H 5850 2700 50  0000 C CNN
 F 1 "FPGA connection" H 5850 600 50  0000 C CNN
-F 2 "Pin_Headers:Pin_Header_Straight_2x20_Pitch2.54mm" H 5800 1700 50  0001 C CNN
+F 2 "Connectors_IDC:IDC-Header_2x20_Pitch2.54mm_Straight" H 5800 1700 50  0001 C CNN
 F 3 "" H 5800 1700 50  0001 C CNN
 	1    5800 1700
@@
 	1    0    0    -1
 $EndComp
+$Comp
+L GND #PWR031
+U 1 1 5A68ECBF
+P 5400 2700
+F 0 "#PWR031" H 5400 2450 50  0001 C CNN
+F 1 "GND" H 5400 2550 50  0000 C CNN
+F 2 "" H 5400 2700 50  0001 C CNN
+F 3 "" H 5400 2700 50  0001 C CNN
+	1    5400 2700
+	0    1    1    0
+$EndComp
 $EndSCHEMATC
