File: rc2014-mystorm.sch (KiCad schematic (older format))
At the start: 26 parts, among them J1 FPGA connection, J2 Config, J3 Conn_01x05, J4 Conn_01x03, J5 Conn_01x05, J6 Extra, P1 RC2014 BUS, U1 SN74LVCC3245A, U2 SN74LVCC3245A, U3 SN74LVCC3245A, U4 SN74LVCC3245A, U5 SN74LVCC3245A, U6 LM1117-3.3

Commit message: gerbers as manuf'd and begginings of hdl
Parts:
- removed J4: Conn_01x03, Pin_Headers:Pin_Header_Straight_1x03_Pitch2.54mm, symbol Conn_01x03
- removed J5: Conn_01x05, Pin_Headers:Pin_Header_Straight_1x05_Pitch2.54mm, symbol Conn_01x05
- C1: value CP_Small -> 100nF
- C2: value CP_Small -> 10uF
- J1: footprint Connectors_IDC:IDC-Header_2x20_Pitch2.54mm_Straight -> Connectors_IDC:IDC-Header_2x25_Pitch2.54mm_Straight; symbol Conn_02x20_Odd_Even -> Conn_02x25_Odd_Even
Connections:
- wire segments 244 -> 246
Other:
- moved on the sheet: U5

Commit message: upgrade to kicad 5, commit of hdl
Parts:
- C1, C2: symbol CP_Small -> Device:CP_Small
- C10, C11, C12, C3, C4, C5, C6, C7, C8, C9: symbol C -> Device:C
- J1: symbol Conn_02x25_Odd_Even -> Connector_Generic:Conn_02x25_Odd_Even
- J2: symbol Conn_02x08_Odd_Even -> Connector_Generic:Conn_02x08_Odd_Even
- J3: symbol Conn_01x04 -> Connector:Conn_01x04_Male
- J6: symbol Conn_01x08 -> Connector:Conn_01x08_Male
- JP1: symbol Jumper_Dual -> Jumper:Jumper_3_Bridged12
- P1: symbol CONN_01X39 -> Connector:Conn_01x39_Male
- U1, U2, U3, U4, U5: symbol SN74LVCC3245A -> rc2014-mystorm:SN74LVCC3245A
- U6: symbol LM1117-3.3 -> rc2014-mystorm-rescue:LM1117-3.3
Connections:
- wire segments 246 -> 284
