File: rc2014-mystorm.kicad_pcb (KiCad board)
At the start: 2 copper layers, 100 x 50 mm, 10 parts, among them J1 CONN_02X06, J2 CONN_02X06, J3 CONN_02X06, J4 CONN_02X17, P1 RC2014 BUS, U1 74HC245, U2 74HC245, U3 74HC245, U4 74HC245, U5 74HC245

Commit message: realise layout blunder
Parts:
- removed U5: 74HC245, Housings_DIP:DIP-20_W7.62mm_Socket
- added J5: CONN_01X10, Pin_Headers:Pin_Header_Straight_1x10_Pitch2.54mm, F.Cu at (110.5, 174.6)
- added J6: CONN_02X06, Pin_Headers:Pin_Header_Straight_2x06_Pitch2.54mm, F.Cu at (155.6, 137.2)
- added J7: CONN_01X06, Pin_Headers:Pin_Header_Straight_1x06_Pitch2.54mm, F.Cu at (135.9, 104.8)
- J4: value CONN_02X17 -> CONN_02X06; footprint Socket_Strips:Socket_Strip_Angled_2x17_Pitch2.54mm -> Pin_Headers:Pin_Header_Straight_2x06_Pitch2.54mm
- U1: value 74HC245 -> 74LVC245
- moved J4 35.1 mm to (158.8, 122.6)
Connections:
- J3 pad 5: /ADDR_DIR -> //RDLV
- J3 pad 6: /ADDR_OE -> //IORQLV
- J4 pad 1: //RDLV -> /ADDR_DIR
- J4 pad 10: /D5LV -> (no net)
- J4 pad 11: /D6LV -> /SIG_OE
- J4 pad 12: /D7LV -> /OE
- J4 pad 2: //IORQLV -> (no net)
- J4 pad 3: /SIG_DIR -> /DATA_DIR
- J4 pad 4: /SIG_OE -> (no net)
- J4 pad 5: /D0LV -> /SIG_DIR
- J4 pad 6: /D1LV -> (no net)
- J4 pad 7: /D2LV -> /ADDR_OE
- J4 pad 8: /D3LV -> /OE
- J4 pad 9: /D4LV -> /DATA_OE
- P1 pad 35: /TX -> (no net)
- P1 pad 36: /RX -> (no net)

Commit message: SMT....
Parts:
- removed J5: CONN_01X10, Pin_Headers:Pin_Header_Straight_1x10_Pitch2.54mm
- added C1: C, Capacitors_SMD:C_1206_HandSoldering, F.Cu at (66.6, 158.8)
- added C2: C, Capacitors_SMD:C_1206_HandSoldering, F.Cu at (89.4, 158.8)
- added C3: C, Capacitors_SMD:C_1206_HandSoldering, F.Cu at (112.3, 158.8)
- added C4: C, Capacitors_SMD:C_1206_HandSoldering, F.Cu at (136.4, 158.8)
- U1: value 74LVC245 -> SN74LVCC3245A; footprint Housings_DIP:DIP-20_W7.62mm_Socket -> Housings_SOIC:SOIC-24W_7.5x15.4mm_Pitch1.27mm
- U2, U3, U4: value 74HC245 -> SN74LVCC3245A; footprint Housings_DIP:DIP-20_W7.62mm_Socket -> Housings_SOIC:SOIC-24W_7.5x15.4mm_Pitch1.27mm
- moved J7 30.5 mm to (153.7, 129.5), turned to 180 degrees
- moved J4 30.4 mm to (132.1, 137.2), turned to 90 degrees
- moved J2 23.3 mm to (78.7, 137.2)
- moved J3 21.7 mm to (105.4, 137.2)
- moved U4 18.8 mm to (141.0, 149.9), turned to 270 degrees
- moved U3 18.7 mm to (118.1, 149.9), turned to 270 degrees
- moved U2 18.2 mm to (95.2, 149.9), turned to 270 degrees
- moved J1 15.3 mm to (64.8, 115.6), turned to 0 degrees
- moved U1 12.2 mm to (73.7, 149.9), turned to 270 degrees
- moved J6 2.62 mm to (156.2, 139.7)
Connections:
- J2 pad 1: GND -> +3V3
- J2 pad 2: GND -> +3V3
- J2 pad 3: +3V3 -> GND
- J2 pad 4: +3V3 -> GND
- J3 pad 1: GND -> +3V3
- J3 pad 2: GND -> +3V3
- J3 pad 3: +3V3 -> GND
- J3 pad 4: +3V3 -> GND
- J6 pad 1: GND -> +3V3
- J6 pad 2: GND -> +3V3
- J6 pad 3: +3V3 -> GND
- J6 pad 4: +3V3 -> GND
- J7 pad 1: GND -> +3V3
- J7 pad 2: +3V3 -> GND
- P1 pad 18: VCC -> +5V
- U1 pad 1: /ADDR_DIR -> +3V3
- U1 pad 10: GND -> /A8LV
- U1 pad 11: /A8LV -> GND
- U1 pad 12: /A9LV -> GND
- U1 pad 13: /A10LV -> GND
- U1 pad 14: /A11LV -> /A15
- U1 pad 15: /A12LV -> /A14
- U1 pad 16: /A13LV -> /A13
- U1 pad 17: /A14LV -> /A12
- U1 pad 18: /A15LV -> /A11
- U1 pad 19: /ADDR_OE -> /A10
- U1 pad 2: /A15 -> /ADDR_DIR
- U1 pad 20: VCC -> /A9
- U1 pad 3: /A14 -> /A15LV
- U1 pad 4: /A13 -> /A14LV
- U1 pad 5: /A12 -> /A13LV
- U1 pad 6: /A11 -> /A12LV
- U1 pad 7: /A10 -> /A11LV
- U1 pad 8: /A9 -> /A10LV
- U1 pad 9: /A8 -> /A9LV
- U2 pad 1: /ADDR_DIR -> +3V3
- U2 pad 10: GND -> /A0LV
- U2 pad 11: /A0LV -> GND
- U2 pad 12: /A1LV -> GND
- U2 pad 13: /A2LV -> GND
- U2 pad 14: /A3LV -> /A7
- U2 pad 15: /A4LV -> /A6
- U2 pad 16: /A5LV -> /A5
- U2 pad 17: /A6LV -> /A4
- U2 pad 18: /A7LV -> /A3
- U2 pad 19: /ADDR_OE -> /A2
- U2 pad 2: /A7 -> /ADDR_DIR
- U2 pad 20: VCC -> /A1
- U2 pad 3: /A6 -> /A7LV
- U2 pad 4: /A5 -> /A6LV
- U2 pad 5: /A4 -> /A5LV
- U2 pad 6: /A3 -> /A4LV
- U2 pad 7: /A2 -> /A3LV
- U2 pad 8: /A1 -> /A2LV
- U2 pad 9: /A0 -> /A1LV
- U3 pad 1: /SIG_DIR -> +3V3
- U3 pad 10: GND -> //IORQLV
- U3 pad 11: //IORQLV -> GND
- U3 pad 12: //RDLV -> GND
- U3 pad 13: //WRLV -> GND
- U3 pad 14: /MREQLV -> /M1
- U3 pad 15: /INTLV -> //RESET
- U3 pad 16: /CLKLV -> /CLK
- U3 pad 17: //RESETLV -> /INT
- U3 pad 18: /M1LV -> /MREQ
- U3 pad 19: /SIG_OE -> //WR
- U3 pad 2: /M1 -> /SIG_DIR
- U3 pad 20: VCC -> //RD
- U3 pad 3: //RESET -> /M1LV
- U3 pad 4: /CLK -> //RESETLV
- U3 pad 5: /INT -> /CLKLV
- U3 pad 6: /MREQ -> /INTLV
- U3 pad 7: //WR -> /MREQLV
- U3 pad 8: //RD -> //WRLV
- U3 pad 9: //IORQ -> //RDLV
- U4 pad 1: /DATA_DIR -> +3V3
- U4 pad 10: GND -> /D7LV
- U4 pad 11: /D7LV -> GND
- U4 pad 12: /D6LV -> GND
- U4 pad 13: /D5LV -> GND
- U4 pad 14: /D4LV -> /D0
- U4 pad 15: /D3LV -> /D1
- U4 pad 16: /D2LV -> /D2
- U4 pad 17: /D1LV -> /D3
- U4 pad 18: /D0LV -> /D4
- U4 pad 19: /DATA_OE -> /D5
- U4 pad 2: /D0 -> /DATA_DIR
- U4 pad 20: VCC -> /D6
- U4 pad 3: /D1 -> /D0LV
- U4 pad 4: /D2 -> /D1LV
- U4 pad 5: /D3 -> /D2LV
- U4 pad 6: /D4 -> /D3LV
- U4 pad 7: /D5 -> /D4LV
- U4 pad 8: /D6 -> /D5LV
- U4 pad 9: /D7 -> /D6LV
Routing:
- net /A7LV: track 40.3 -> 0.00 mm
- net /A6LV: track 31.5 -> 0.00 mm
- net /A5LV: track 30.9 -> 0.00 mm
- net /A4LV: track 30.4 -> 0.00 mm
- net /A15LV: track 24.0 -> 0.00 mm
- net /A8: track 22.5 -> 0.00 mm
- net /A9: track 21.1 -> 0.00 mm
- net /INT: track 20.9 -> 0.00 mm
- net //WR: track 20.9 -> 0.00 mm
- net //RESET: track 20.9 -> 0.00 mm
- net /MREQ: track 20.9 -> 0.00 mm
- net /M1: track 20.9 -> 0.00 mm
- net /CLK: track 20.9 -> 0.00 mm
- net //RD: track 20.9 -> 0.00 mm
- net //IORQ: track 20.9 -> 0.00 mm
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
Commit message: further SMT WIP
Parts:
- removed J7: CONN_01X06, Pin_Headers:Pin_Header_Straight_1x06_Pitch2.54mm
- added C10: C, Capacitors_SMD:C_0805_HandSoldering, B.Cu at (117.5, 149.9)
- added C11: C, Capacitors_SMD:C_0805_HandSoldering, B.Cu at (137.8, 149.9)
- added C12: C, Capacitors_SMD:C_0805_HandSoldering, B.Cu at (158.1, 149.9)
- added C5: C, Capacitors_SMD:C_0805_HandSoldering, B.Cu at (113.7, 149.8)
- added C6: C, Capacitors_SMD:C_0805_HandSoldering, B.Cu at (134.0, 149.8)
- added C7: C, Capacitors_SMD:C_0805_HandSoldering, B.Cu at (154.3, 149.8)
- added C8: C, Capacitors_SMD:C_0805_HandSoldering, B.Cu at (76.8, 149.9)
- added C9: C, Capacitors_SMD:C_0805_HandSoldering, B.Cu at (97.2, 149.9)
- added J5: Conn_01x05, Pin_Headers:Pin_Header_Straight_1x05_Pitch2.54mm, F.Cu at (104.1, 139.7)
- added JP1: Ext Power, Pin_Headers:Pin_Header_Straight_1x03_Pitch2.54mm, F.Cu at (80.6, 141.6)
- added U5: SN74LVCC3245A, Housings_SOIC:SOIC-24W_7.5x15.4mm_Pitch1.27mm, F.Cu at (151.1, 149.9)
- added U6: LM1117-3.3, TO_SOT_Packages_SMD:SOT-223-3_TabPin2, B.Cu at (73.7, 141.6)
- C1, C2: value C -> CP_Small; footprint Capacitors_SMD:C_1206_HandSoldering -> Capacitors_SMD:C_0805_HandSoldering; moved to B.Cu
- C3, C4: footprint Capacitors_SMD:C_1206_HandSoldering -> Capacitors_SMD:C_0805_HandSoldering; moved to B.Cu
- J1: value CONN_02X06 -> FPGA connection; footprint Pin_Headers:Pin_Header_Straight_2x06_Pitch2.54mm -> Pin_Headers:Pin_Header_Straight_2x20_Pitch2.54mm
- J2: value CONN_02X06 -> Config; footprint Pin_Headers:Pin_Header_Straight_2x06_Pitch2.54mm -> Pin_Headers:Pin_Header_Straight_2x08_Pitch2.54mm
- J3: value CONN_02X06 -> Conn_01x05; footprint Pin_Headers:Pin_Header_Straight_2x06_Pitch2.54mm -> Pin_Headers:Pin_Header_Straight_1x04_Pitch2.54mm
- J4: value CONN_02X06 -> Conn_01x03; footprint Pin_Headers:Pin_Header_Straight_2x06_Pitch2.54mm -> Pin_Headers:Pin_Header_Straight_1x03_Pitch2.54mm
- J6: value CONN_02X06 -> Extra; footprint Pin_Headers:Pin_Header_Straight_2x06_Pitch2.54mm -> Pin_Headers:Pin_Header_Straight_1x08_Pitch2.54mm
- moved J2 61.0 mm to (139.7, 134.0)
- moved J3 44.5 mm to (149.9, 136.5)
- moved C4 44.0 mm to (93.3, 149.8), turned to 270 degrees
- moved C3 40.3 mm to (73.0, 149.9), turned to 270 degrees
- moved J6 34.5 mm to (128.3, 160.0), turned to 90 degrees
- moved U4 30.5 mm to (110.5, 149.9)
- moved J1 27.4 mm to (85.1, 134.0), turned to 90 degrees
- moved C2 22.5 mm to (81.3, 137.8)
- moved C1 15.2 mm to (66.7, 143.5)
- moved U3 12.7 mm to (130.8, 149.9)
- moved J4 9.38 mm to (123.8, 141.6)
- moved U2 5.08 mm to (90.2, 149.9)
- moved U1 3.81 mm to (69.8, 149.9)
- moved P1 0.23 mm to (62.2, 163.0)
Connections:
- C1 pad 1: (no net) -> +5V
- C2 pad 1: (no net) -> Net-(C2-Pad1)
- C2 pad 2: (no net) -> GND
- C3 pad 1: (no net) -> +3V3
- C3 pad 2: (no net) -> GND
- C4 pad 1: (no net) -> +3V3
- C4 pad 2: (no net) -> GND
- J1 pad 1: GND -> /FPGA_VCC
- J1 pad 10: /A11LV -> /A9LV
- J1 pad 11: /A8LV -> /A6LV
- J1 pad 12: /A9LV -> /A7LV
- J1 pad 3: +3V3 -> /A14LV
- J1 pad 4: +3V3 -> /A15LV
- J1 pad 5: /A14LV -> /A12LV
- J1 pad 6: /A15LV -> /A13LV
- J1 pad 7: /A12LV -> /A10LV
- J1 pad 8: /A13LV -> /A11LV
- J1 pad 9: /A10LV -> /A8LV
- J2 pad 1: +3V3 -> /ADDR_DIR
- J2 pad 10: /A3LV -> GND
- J2 pad 11: /A0LV -> /DATA_OE
- J2 pad 12: /A1LV -> GND
- J2 pad 2: +3V3 -> /GPIO1
- J2 pad 3: GND -> /DATA_DIR
- J2 pad 4: GND -> /GPIO2
- J2 pad 5: /A6LV -> /SIG_DIR
- J2 pad 6: /A7LV -> /GPIO3
- J2 pad 7: /A4LV -> /SIG2_DIR
- J2 pad 8: /A5LV -> /GPIO4
- J2 pad 9: /A2LV -> /ADDR_OE
- J3 pad 3: GND -> +3V3
- J3 pad 4: GND -> +3V3
- J4 pad 1: /ADDR_DIR -> /EX3LV
- J4 pad 2: (no net) -> /EX2LV
- J4 pad 3: /DATA_DIR -> /EX1LV
- J6 pad 1: +3V3 -> /EX8
- J6 pad 2: +3V3 -> /EX7
- J6 pad 3: GND -> /EX6
- J6 pad 4: GND -> /EX5
- J6 pad 5: /D0LV -> /EX4
- J6 pad 6: /D1LV -> /EX3
- J6 pad 7: /D2LV -> /EX2
- J6 pad 8: /D3LV -> /EX1
- U1 pad 10: /A8LV -> /A15LV
- U1 pad 3: /A15LV -> /A8LV
- U1 pad 4: /A14LV -> /A9LV
- U1 pad 5: /A13LV -> /A10LV
- U1 pad 6: /A12LV -> /A11LV
- U1 pad 7: /A11LV -> /A12LV
- U1 pad 8: /A10LV -> /A13LV
- U1 pad 9: /A9LV -> /A14LV
- U2 pad 10: /A0LV -> /A7LV
- U2 pad 3: /A7LV -> /A0LV
- U2 pad 4: /A6LV -> /A1LV
- U2 pad 5: /A5LV -> /A2LV
- U2 pad 6: /A4LV -> /A3LV
- U2 pad 7: /A3LV -> /A4LV
- U2 pad 8: /A2LV -> /A5LV
- U2 pad 9: /A1LV -> /A6LV
- U3 pad 10: //IORQLV -> /EX3LV
- U3 pad 14: /M1 -> /EX3
- U3 pad 15: //RESET -> /EX2
- U3 pad 16: /CLK -> /EX1
- U3 pad 17: /INT -> /M1
- U3 pad 3: /M1LV -> //IORQLV
- U3 pad 4: //RESETLV -> //RDLV
- U3 pad 5: /CLKLV -> //WRLV
- U3 pad 6: /INTLV -> /MREQLV
- U3 pad 7: /MREQLV -> /M1LV
- U3 pad 8: //WRLV -> /EX1LV
- U3 pad 9: //RDLV -> /EX2LV
- U4 pad 10: /D7LV -> /EX8LV
- U4 pad 14: /D0 -> /EX8
- U4 pad 15: /D1 -> /EX7
- U4 pad 16: /D2 -> /EX6
- U4 pad 17: /D3 -> /EX5
- U4 pad 18: /D4 -> /EX4
- U4 pad 19: /D5 -> //RESET
- U4 pad 2: /DATA_DIR -> /SIG2_DIR
- U4 pad 20: /D6 -> /CLK
- U4 pad 21: /D7 -> /INT
- U4 pad 22: /DATA_OE -> /SIG2_OE
- U4 pad 3: /D0LV -> /INTLV
- U4 pad 4: /D1LV -> /CLKLV
- U4 pad 5: /D2LV -> //RESETLV
- U4 pad 6: /D3LV -> /EX4LV
- U4 pad 7: /D4LV -> /EX5LV
- U4 pad 8: /D5LV -> /EX6LV
- U4 pad 9: /D6LV -> /EX7LV
Routing:
- net GND: track 0.00 -> 263.6 mm, vias 0 -> 12
- net +5V: track 0.00 -> 132.2 mm, vias 0 -> 6
- net +3V3: track 0.00 -> 132.1 mm, vias 0 -> 5
- net /ADDR_OE: track 0.00 -> 89.8 mm, vias 0 -> 1
- net /ADDR_DIR: track 0.00 -> 74.3 mm, vias 0 -> 1
- net /SIG2_OE: track 0.00 -> 55.6 mm, vias 0 -> 1
- net //IORQLV: track 0.00 -> 38.5 mm, vias 0 -> 2
- net /D3LV: track 0.00 -> 37.1 mm
- net /D1LV: track 0.00 -> 37.0 mm
- net /D5LV: track 0.00 -> 37.0 mm
- net /SIG2_DIR: track 0.00 -> 36.8 mm, vias 0 -> 1
- net //RDLV: track 0.00 -> 36.8 mm, vias 0 -> 2
- net /D7LV: track 0.00 -> 35.9 mm
- net /D0LV: track 0.00 -> 34.4 mm
- net /D4LV: track 0.00 -> 34.3 mm
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Other:
- outline, holes or cut-outs redrawn
- net class Default: clearance 0.254 -> 0.2
- rule trace_clearance: 0.254 -> 0.2
- board text added: "A15"
- board text added: "github.com/electrified/rc2014-fpga"
- board text removed: "github.com/electrified/rc2014-ym2149"

Commit message: WIP
Parts:
- added REF***: OSHW-Logo_7.5x8mm_SilkScreen, Symbols:OSHW-Logo_7.5x8mm_SilkScreen, B.Cu at (71.1, 125.7)
- J1: footprint Pin_Headers:Pin_Header_Straight_2x20_Pitch2.54mm -> Connectors_IDC:IDC-Header_2x20_Pitch2.54mm_Straight
- moved C2 9.86 mm to (71.8, 140.3)
- moved J1 9.25 mm to (82.5, 125.1)
- moved J2 8.89 mm to (139.7, 125.1)
- moved J3 8.89 mm to (149.9, 127.6)
- moved U6 8.47 mm to (65.4, 143.5)
- moved C1 7.10 mm to (65.4, 150.5)
- moved J4 5.24 mm to (125.1, 136.5)
- moved JP1 5.08 mm to (80.6, 136.5)
- moved J5 3.24 mm to (104.8, 136.5)
- moved C10 2.54 mm to (117.5, 147.3)
- moved C11 2.54 mm to (137.8, 147.3)
- moved C12 2.54 mm to (158.1, 147.3)
- moved C3 2.54 mm to (73.0, 147.3)
- moved C8 2.54 mm to (76.8, 147.3)
- moved C9 2.54 mm to (97.2, 147.3)
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Connections:
- J1 pad 39: /FPGA_VCC -> GND
Routing:
- net /ADDR_OE: track 89.8 -> 25.3 mm, vias 1 -> 0
- net /SIG2_OE: track 55.6 -> 0.00 mm, vias 1 -> 0
- net GND: track 263.6 -> 315.0 mm
- net /ADDR_DIR: track 74.3 -> 26.6 mm, vias 1 -> 0
- net /SIG2_DIR: track 36.8 -> 1.37 mm, vias 1 -> 0
- net /EX4: track 31.8 -> 0.00 mm, vias 1 -> 0
- net /SIG_OE: track 31.6 -> 0.00 mm, vias 1 -> 0
- net /EX5: track 31.0 -> 0.00 mm, vias 1 -> 0
- net /EX6: track 29.9 -> 0.00 mm, vias 1 -> 0
- net /EX7: track 28.9 -> 0.00 mm, vias 1 -> 0
- net /EX8: track 28.0 -> 0.00 mm, vias 1 -> 0
- net /M1LV: track 27.2 -> 0.00 mm
- net /M1: track 26.3 -> 0.00 mm, vias 1 -> 0
- net //WRLV: track 25.6 -> 0.14 mm
- net /DATA_OE: track 24.6 -> 0.70 mm
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- added copper zone on B.Cu, net GND
Other:
- outline, holes or cut-outs redrawn
- net class IO: clearance 0.254 -> 0.2
- net class analogue: clearance 0.254 -> 0.2
- net class gnd: clearance 0.254 -> 0.2
- net class vcc: clearance 0.254 -> 0.2
- board text added: "+3.3V"
- board text added: "+5V"
- board text added: "3.3V source"
- board text added: "A0"
- board text added: "A1"
- board text added: "A10"
- board text added: "A11"
- board text added: "A12"
- board text added: "A13"
- board text added: "A14"
- board text added: "A2"
- board text added: "A3"
- board text added: "A4"
- board text added: "A5"
- board text added: "A6"
- board text added: "A7"
- board text added: "A8"
- board text added: "A9"
- board text added: "ADDR"
- board text added: "CLK"
- board text added: "D0"
- board text added: "D1"
- board text added: "D2"
- board text added: "D3"
- board text added: "D4"
- board text added: "D5"
- board text added: "D6"
- board text added: "D7"
- board text added: "DATA"
- board text added: "DIR"
- board text added: "FPGA"
- board text added: "G1"
- board text added: "G2"
- board text added: "G3"
- board text added: "G4"
- board text added: "GND"
- board text added: "INT"
- board text added: "IORQ"
- board text added: "M1"
- board text added: "MRQ"
- board text added: "OE"
- board text added: "R1"
- board text added: "RC2014 5V <-> 3.3V FPGA Interface"
- board text added: "RD"
- board text added: "RST"
- board text added: "Reg"
- board text added: "SIG"
- board text added: "SIG2"
- board text added: "WR"
- board text added: "github.com/electrified/rc2014-fpga-interface"
- board text removed: "github.com/electrified/rc2014-fpga"

Commit message: gerbers as manuf'd and begginings of hdl
Parts:
- removed J4: Conn_01x03, Pin_Headers:Pin_Header_Straight_1x03_Pitch2.54mm
- removed J5: Conn_01x05, Pin_Headers:Pin_Header_Straight_1x05_Pitch2.54mm
- removed the REF*** at (71.1, 125.7)
- added REF***: OSHW-Logo2_14.6x12mm_SilkScreen, Symbols:OSHW-Logo2_14.6x12mm_SilkScreen, B.Cu at (146.7, 154.3)
- J1: footprint Connectors_IDC:IDC-Header_2x20_Pitch2.54mm_Straight -> Connectors_IDC:IDC-Header_2x25_Pitch2.54mm_Straight
- moved J6 20.3 mm to (108.0, 160.7)
- moved J2 14.9 mm to (153.2, 118.7), turned to 0 degrees
- moved JP1 14.0 mm to (69.8, 127.6), turned to 0 degrees
- moved J1 2.54 mm to (80.0, 125.1)
- moved J3 1.44 mm to (150.7, 128.8), turned to 0 degrees
Connections:
- J1 pad 19: //RDLV -> /M1LV
- J1 pad 21: /M1LV -> //RDLV
- J1 pad 39: GND -> /EX8LV
- J1 pad 40: GND -> /EX7LV
Routing:
- net GND: track 315.0 -> 234.5 mm, vias 12 -> 8
- net /ADDR_DIR: track 26.6 -> 101.7 mm
- net /ADDR_OE: track 25.3 -> 95.4 mm, vias 0 -> 1
- net /SIG2_OE: track 0.00 -> 47.3 mm, vias 0 -> 1
- net /SIG2_DIR: track 1.37 -> 44.6 mm, vias 0 -> 1
- net //WRLV: track 0.14 -> 36.2 mm
- net /M1LV: track 0.00 -> 36.0 mm, vias 0 -> 1
- net /M1: track 0.00 -> 34.2 mm, vias 0 -> 1
- net /MREQLV: track 0.70 -> 32.6 mm
- net /SIG_OE: track 0.00 -> 29.7 mm, vias 0 -> 1
- net /GPIO1: track 16.5 -> 43.9 mm
- net /SIG_DIR: track 0.00 -> 26.8 mm, vias 0 -> 1
- net /EX7LV: track 6.09 -> 32.1 mm, vias 0 -> 1
- net /EX5LV: track 7.15 -> 32.8 mm, vias 0 -> 1
- net /EX6LV: track 6.62 -> 31.8 mm, vias 0 -> 1
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Other:
- board text added: "2018 Ed Brindley"
- board text added: "EX1"
- board text added: "EX2"
- board text added: "EX3"
- board text added: "EX4"
- board text added: "EX5"
- board text added: "EX6"
- board text added: "EX7"
- board text added: "EX8"
- board text added: "Rev 1"
- board text removed: "R1"
