File: rc2014-mystorm.kicad_pcb (KiCad board)
At the start: 2 copper layers, 100 x 50 mm, 25 parts, among them J1 FPGA connection, J2 Config, J3 Conn_01x05, J6 Extra, P1 RC2014 BUS, U1 SN74LVCC3245A, U2 SN74LVCC3245A, U3 SN74LVCC3245A, U4 SN74LVCC3245A, U5 SN74LVCC3245A, U6 LM1117-3.3

Commit message: convert to nextpnr
Parts:
- C1: value CP_Small -> 100nF
- C2: value CP_Small -> 10uF
Connections:
- P1 pad 35: (no net) -> /TX
- P1 pad 36: (no net) -> /RX
- P1 pad 37: (no net) -> Net-(P1-Pad37)
- P1 pad 38: (no net) -> Net-(P1-Pad38)
- P1 pad 39: (no net) -> Net-(P1-Pad39)
- U1 pad 23: (no net) -> Net-(U1-Pad23)
- U2 pad 23: (no net) -> Net-(U2-Pad23)
- U3 pad 23: (no net) -> Net-(U3-Pad23)
- U4 pad 23: (no net) -> Net-(U4-Pad23)
- U5 pad 23: (no net) -> Net-(U5-Pad23)
Changed lines of the file:
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@@
     (zones 0)
     (modules 25)
-    (nets 98)
+    (nets 108)
   )
   (page A4)
@@
   (net 96 /CLK)
   (net 97 /INT)
+  (net 98 /TX)
+  (net 99 /RX)
+  (net 100 "Net-(P1-Pad37)")
+  (net 101 "Net-(P1-Pad38)")
+  (net 102 "Net-(P1-Pad39)")
+  (net 103 "Net-(U1-Pad23)")
+  (net 104 "Net-(U2-Pad23)")
+  (net 105 "Net-(U3-Pad23)")
+  (net 106 "Net-(U4-Pad23)")
+  (net 107 "Net-(U5-Pad23)")
   (net_class Default "This is the default net class."
     (clearance 0.2)
@@
     (add_net /MREQ)
     (add_net /MREQLV)
+    (add_net /RX)
     (add_net /SIG2_DIR)
     (add_net /SIG2_OE)
     (add_net /SIG_DIR)
     (add_net /SIG_OE)
+    (add_net /TX)
     (add_net "Net-(C2-Pad1)")
+    (add_net "Net-(P1-Pad37)")
+    (add_net "Net-(P1-Pad38)")
+    (add_net "Net-(P1-Pad39)")
+    (add_net "Net-(U1-Pad23)")
+    (add_net "Net-(U2-Pad23)")
+    (add_net "Net-(U3-Pad23)")
+    (add_net "Net-(U4-Pad23)")
+    (add_net "Net-(U5-Pad23)")
   )
   (net_class IO ""
@@
     (pad 22 smd rect (at 4.7 -4.445 270) (size 2 0.6) (layers F.Cu F.Paste F.Mask)
       (net 68 /DATA_OE))
-    (pad 23 smd rect (at 4.7 -5.715 270) (size 2 0.6) (layers F.Cu F.Paste F.Mask))
+    (pad 23 smd rect (at 4.7 -5.715 270) (size 2 0.6) (layers F.Cu F.Paste F.Mask)
+      (net 107 "Net-(U5-Pad23)"))
     (pad 24 smd rect (at 4.7 -6.985 270) (size 2 0.6) (layers F.Cu F.Paste F.Mask)
       (net 69 +5V))
@@
     (pad 22 smd rect (at 4.7 -4.445 270) (size 2 0.6) (layers F.Cu F.Paste F.Mask)
       (net 65 /ADDR_OE))
-    (pad 23 smd rect (at 4.7 -5.715 270) (size 2 0.6) (layers F.Cu F.Paste F.Mask))
+    (pad 23 smd rect (at 4.7 -5.715 270) (size 2 0.6) (layers F.Cu F.Paste F.Mask)
+      (net 104 "Net-(U2-Pad23)"))
     (pad 24 smd rect (at 4.7 -6.985 270) (size 2 0.6) (layers F.Cu F.Paste F.Mask)
       (net 69 +5V))
@@
     (pad 22 smd rect (at 4.7 -4.445 270) (size 2 0.6) (layers F.Cu F.Paste F.Mask)
       (net 67 /SIG_OE))
-    (pad 23 smd rect (at 4.7 -5.715 270) (size 2 0.6) (layers F.Cu F.Paste F.Mask))
+    (pad 23 smd rect (at 4.7 -5.715 270) (size 2 0.6) (layers F.Cu F.Paste F.Mask)
+      (net 105 "Net-(U3-Pad23)"))
     (pad 24 smd rect (at 4.7 -6.985 270) (size 2 0.6) (layers F.Cu F.Paste F.Mask)
       (net 69 +5V))
@@
     (pad 22 smd rect (at 4.7 -4.445 270) (size 2 0.6) (layers F.Cu F.Paste F.Mask)
       (net 77 /SIG2_OE))
-    (pad 23 smd rect (at 4.7 -5.715 270) (size 2 0.6) (layers F.Cu F.Paste F.Mask))
+    (pad 23 smd rect (at 4.7 -5.715 270) (size 2 0.6) (layers F.Cu F.Paste F.Mask)
+      (net 106 "Net-(U4-Pad23)"))
     (pad 24 smd rect (at 4.7 -6.985 270) (size 2 0.6) (layers F.Cu F.Paste F.Mask)
       (net 69 +5V))
@@
     (pad 34 thru_hole oval (at 0 83.82 90) (size 2 2) (drill 1) (layers *.Cu *.Mask)
       (net 11 /D7))
-    (pad 35 thru_hole oval (at 0 86.36 90) (size 2 2) (drill 1) (layers *.Cu *.Mask))
-    (pad 36 thru_hole oval (at 0 88.9 90) (size 2 2) (drill 1) (layers *.Cu *.Mask))
-    (pad 37 thru_hole oval (at 0 91.44 90) (size 2 2) (drill 1) (layers *.Cu *.Mask))
-    (pad 38 thru_hole oval (at 0 93.98 90) (size 2 2) (drill 1) (layers *.Cu *.Mask))
-    (pad 39 thru_hole oval (at 0 96.52 90) (size 2 2) (drill 1) (layers *.Cu *.Mask))
+    (pad 35 thru_hole oval (at 0 86.36 90) (size 2 2) (drill 1) (layers *.Cu *.Mask)
+      (net 98 /TX))
+    (pad 36 thru_hole oval (at 0 88.9 90) (size 2 2) (drill 1) (layers *.Cu *.Mask)
+      (net 99 /RX))
+    (pad 37 thru_hole oval (at 0 91.44 90) (size 2 2) (drill 1) (layers *.Cu *.Mask)
+      (net 100 "Net-(P1-Pad37)"))
+    (pad 38 thru_hole oval (at 0 93.98 90) (size 2 2) (drill 1) (layers *.Cu *.Mask)
+      (net 101 "Net-(P1-Pad38)"))
+    (pad 39 thru_hole oval (at 0 96.52 90) (size 2 2) (drill 1) (layers *.Cu *.Mask)
+      (net 102 "Net-(P1-Pad39)"))
     (model ${KISYS3DMOD}/Pin_Headers.3dshapes/Pin_Header_Straight_1x39_Pitch2.54mm.wrl
       (offset (xyz 0 -48.25999927520752 0))
@@
     (pad 22 smd rect (at 4.7 -4.445 270) (size 2 0.6) (layers F.Cu F.Paste F.Mask)
       (net 65 /ADDR_OE))
-    (pad 23 smd rect (at 4.7 -5.715 270) (size 2 0.6) (layers F.Cu F.Paste F.Mask))
+    (pad 23 smd rect (at 4.7 -5.715 270) (size 2 0.6) (layers F.Cu F.Paste F.Mask)
+      (net 103 "Net-(U1-Pad23)"))
     (pad 24 smd rect (at 4.7 -6.985 270) (size 2 0.6) (layers F.Cu F.Paste F.Mask)
       (net 69 +5V))
@@
       (effects (font (size 1 1) (thickness 0.2)) (justify mirror))
     )
-    (fp_text value CP_Small (at 0 -1.75) (layer B.Fab)
+    (fp_text value 100nF (at 0 -1.75) (layer B.Fab)
       (effects (font (size 1 1) (thickness 0.15)) (justify mirror))
     )
@@
       (effects (font (size 1 1) (thickness 0.2)) (justify mirror))
     )
-    (fp_text value CP_Small (at 0 -1.75) (layer B.Fab)
+    (fp_text value 10uF (at 0 -1.75) (layer B.Fab)
       (effects (font (size 1 1) (thickness 0.15)) (justify mirror))
     )

Commit message: resave with kicad 9 and tidy up - no attempt made to update to new component libraries
Connections:
- net +3V3 renamed +3.3V
- net //IORQ renamed //IORQ
- net //IORQLV renamed //IORQLV
- net //RD renamed //RD
- net //RDLV renamed //RDLV
- net //RESET renamed //RESET
- net //RESETLV renamed //RESETLV
- net //WR renamed //WR
- net //WRLV renamed //WRLV
- P1 pad 37: Net-(P1-Pad37) -> unconnected-(P1-Pin_37-Pad37)
- P1 pad 38: Net-(P1-Pad38) -> unconnected-(P1-Pin_38-Pad38)
- P1 pad 39: Net-(P1-Pad39) -> unconnected-(P1-Pin_39-Pad39)
- U1 pad 23: Net-(U1-Pad23) -> unconnected-(U1-NC-Pad23)
- U2 pad 23: Net-(U2-Pad23) -> unconnected-(U2-NC-Pad23)
- U3 pad 23: Net-(U3-Pad23) -> unconnected-(U3-NC-Pad23)
- U4 pad 23: Net-(U4-Pad23) -> unconnected-(U4-NC-Pad23)
- U5 pad 23: Net-(U5-Pad23) -> unconnected-(U5-NC-Pad23)
Other:
- net class Default removed
- net class IO removed
- net class analogue removed
- net class gnd removed
- net class vcc removed
